Commit message: FIX: Fixed swerve driver

File: webots_tutotrial_1/install/webots_pkg_sim/share/webots_pkg_sim/urdf/new_rover.urdf (robot description, URDF)
Before this commit: robot new_rover, 11 links, 10 joints
Links:
- removed link oakd_optical_link
- added link gps_link, mass 0.01; visual box size=0.05 0.05 0.02
- added link imu_link, mass 0.01
- added link oakd_depth_optical_link
- added link oakd_rgb_optical_link
Joints:
- removed joint oakd_optical_joint
- added joint gps_joint: type fixed, parent base_link, child gps_link, origin xyz=0 0 0.22 rpy=0 0 0
- added joint imu_joint: type fixed, parent base_link, child imu_link, origin xyz=0 0 0.1 rpy=0 0 0
- added joint oakd_depth_optical_joint: type fixed, parent oakd_link, child oakd_depth_optical_link, origin xyz=0 0 0 rpy=-1.5708 0 -1.5708
- added joint oakd_rgb_optical_joint: type fixed, parent oakd_link, child oakd_rgb_optical_link, origin xyz=0 0 0 rpy=-1.5708 0 -1.5708
